File: lang1.kicad_pcb (KiCad board)
At the start: 2 copper layers, 76.6 x 25.4 mm, 18 parts, among them J1 Conn_01x04, J2 Conn_01x04, J3 Conn_01x02_Pin, U1 ADS1115IDGS

Commit message: senger
Parts:
- H1, H2, H3, H4: footprint MountingHole:MountingHole_3.2mm_M3 -> MountingHole:MountingHole_3.2mm_M3_DIN965_Pad
- J3: footprint Connector_PinHeader_1.27mm:PinHeader_1x02_P1.27mm_Vertical -> Connector_PinHeader_2.54mm:PinHeader_1x02_P2.54mm_Vertical
- moved J3 4.80 mm to (123.4, 59.5), turned to 90 degrees
- moved R1 3.59 mm to (122.7, 62.0)
- moved ADS1115IDGS 0.16 mm to (130.7, 63.1)
- renumbered U1 to ADS1115IDGS
Connections:
- C1 pad 1: GND -> /GND2
- FB1 pad 2: GND -> /GND2
- J1 pad 2: GND -> /GND2
- J2 pad 2: GND -> /GND2
- VDD pad 2: GND -> /GND2 (x2)
Routing:
- net GND: track 116.7 -> 11.1 mm, vias 6 -> 3
- net /GND2: track 0.00 -> 81.1 mm, vias 0 -> 3
- net Net-(J3-Pin_1): track 9.84 -> 14.4 mm
- net Net-(J3-Pin_2): track 17.6 -> 15.2 mm
- added copper zone on B.Cu, net GND
Other:
- board text added: "ADDR"
- board text added: "GND"
- board text added: "RDY"
- board text added: "SCL"
- board text added: "SDA"
- board text added: "VDD"
